File: hardware/batteryTester.kicad_pcb (KiCad board)
At the start: 2 copper layers, 45 x 105 mm, 45 parts, among them J1 OLED_DISPLAY, J2 USB_C_Receptacle_USB2.0_16P, J3 PROG, Q1 IRF540N, SW1 START, SW2 STOP, SW3 STOP, U1 AMS1117-3.3, U2 LMV321, U3 LMV321, U4 ATSAMD21E15B-A, Y1 32.768kHz

Commit message: code runs!
Parts:
- added J1: OLED_DISPLAY, Connector_PinSocket_2.54mm:PinSocket_1x04_P2.54mm_Vertical, F.Cu at (155.1, 128.3)
